File: dac_sch.kicad_sch (KiCad schematic)
At the start: 17 parts

Commit message: ERC valid.
Parts:
- gave numbers to parts that had none: 17
Connections:
- net SPI2_SCLK renamed SPI2_SCK
Other:
- moved on the sheet: C401

Commit message: Assigned Footprints and Set up board specifications.
Parts:
- C400, C402, C403, C404, C405: footprint (none) -> Capacitor_SMD:C_0402_1005Metric
- C401, C406: footprint (none) -> Capacitor_SMD:C_0603_1608Metric
- D400: footprint (none) -> Diode_SMD:D_SOD-323
- J400: footprint (none) -> Connector_Coaxial:BNC_Amphenol_031-6575_Horizontal
- R400, R401, R402, R403, R404, R405: footprint (none) -> Resistor_SMD:R_0402_1005Metric
- U401: footprint (none) -> my_footprints:SOIC-10
Changed lines of the file:
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@@
     (property "Reference" "R403" (id 0) (at 196.85 57.785 90))
     (property "Value" "49R9" (id 1) (at 196.85 61.595 90))
-    (property "Footprint" "" (id 2) (at 196.85 57.912 90)
+    (property "Footprint" "Resistor_SMD:R_0402_1005Metric" (id 2) (at 196.85 57.912 90)
       (effects (font (size 1.27 1.27)) hide)
     )
@@
     (property "Reference" "R402" (id 0) (at 146.05 55.245 90))
     (property "Value" "12k" (id 1) (at 146.05 59.055 90))
-    (property "Footprint" "" (id 2) (at 146.05 55.372 90)
+    (property "Footprint" "Resistor_SMD:R_0402_1005Metric" (id 2) (at 146.05 55.372 90)
       (effects (font (size 1.27 1.27)) hide)
     )
@@
       (effects (font (size 1.27 1.27)) (justify left))
     )
-    (property "Footprint" "" (id 2) (at 95.885 71.755 0)
+    (property "Footprint" "Capacitor_SMD:C_0603_1608Metric" (id 2) (at 95.885 71.755 0)
       (effects (font (size 1.27 1.27)) hide)
     )
@@
       (effects (font (size 1.27 1.27)) (justify left))
     )
-    (property "Footprint" "" (id 2) (at 105.537 72.39 90)
+    (property "Footprint" "Resistor_SMD:R_0402_1005Metric" (id 2) (at 105.537 72.39 90)
       (effects (font (size 1.27 1.27)) hide)
     )
@@
     (property "Reference" "C404" (id 0) (at 130.175 62.23 0))
     (property "Value" "1n" (id 1) (at 128.905 64.77 0))
-    (property "Footprint" "" (id 2) (at 125.73 62.865 0)
+    (property "Footprint" "Capacitor_SMD:C_0402_1005Metric" (id 2) (at 125.73 62.865 0)
       (effects (font (size 1.27 1.27)) hide)
     )
@@
       (effects (font (size 1.27 1.27)) (justify left))
     )
-    (property "Footprint" "" (id 2) (at 66.04 47.625 0)
+    (property "Footprint" "Capacitor_SMD:C_0402_1005Metric" (id 2) (at 66.04 47.625 0)
       (effects (font (size 1.27 1.27)) hide)
     )
@@
     (property "Reference" "R400" (id 0) (at 118.745 55.245 90))
     (property "Value" "6k8" (id 1) (at 118.745 59.055 90))
-    (property "Footprint" "" (id 2) (at 118.745 55.372 90)
+    (property "Footprint" "Resistor_SMD:R_0402_1005Metric" (id 2) (at 118.745 55.372 90)
       (effects (font (size 1.27 1.27)) hide)
     )
@@
       (effects (font (size 1.27 1.27)) (justify right))
     )
-    (property "Footprint" "" (id 2) (at 207.01 66.04 0)
+    (property "Footprint" "Diode_SMD:D_SOD-323" (id 2) (at 207.01 66.04 0)
       (effects (font (size 1.27 1.27)) hide)
     )
@@
     (property "Reference" "C403" (id 0) (at 161.29 45.085 90))
     (property "Value" "100n" (id 1) (at 161.29 47.625 90))
-    (property "Footprint" "" (id 2) (at 161.29 50.8 0)
+    (property "Footprint" "Capacitor_SMD:C_0402_1005Metric" (id 2) (at 161.29 50.8 0)
       (effects (font (size 1.27 1.27)) hide)
     )
@@
       (effects (font (size 1.27 1.27)) (justify left))
     )
-    (property "Footprint" "" (id 2) (at 55.88 47.625 0)
+    (property "Footprint" "Capacitor_SMD:C_0603_1608Metric" (id 2) (at 55.88 47.625 0)
       (effects (font (size 1.27 1.27)) hide)
     )
@@
     (property "Reference" "C405" (id 0) (at 156.21 60.96 0))
     (property "Value" "150p" (id 1) (at 156.21 64.77 0))
-    (property "Footprint" "" (id 2) (at 153.035 62.865 0)
+    (property "Footprint" "Capacitor_SMD:C_0402_1005Metric" (id 2) (at 153.035 62.865 0)
       (effects (font (size 1.27 1.27)) hide)
     )
@@
       (effects (font (size 1.27 1.27)) (justify left))
     )
-    (property "Footprint" "" (id 2) (at 78.74 57.15 0)
+    (property "Footprint" "my_footprints:SOIC-10" (id 2) (at 78.74 57.15 0)
       (effects (font (size 1.27 1.27)) hide)
     )
@@
     (property "Reference" "R404" (id 0) (at 51.435 62.865 90))
     (property "Value" "0R" (id 1) (at 51.435 60.96 90))
-    (property "Footprint" "" (id 2) (at 51.435 62.738 90)
+    (property "Footprint" "Resistor_SMD:R_0402_1005Metric" (id 2) (at 51.435 62.738 90)
       (effects (font (size 1.27 1.27)) hide)
     )
@@
     (property "Reference" "J400" (id 0) (at 220.98 55.88 0))
     (property "Value" "DOSIN-801-0031" (id 1) (at 224.79 59.69 90))
-    (property "Footprint" "" (id 2) (at 220.98 59.69 0)
+    (property "Footprint" "Connector_Coaxial:BNC_Amphenol_031-6575_Horizontal" (id 2) (at 220.98 59.69 0)
       (effects (font (size 1.27 1.27)) hide)
     )
@@
     (property "Reference" "C400" (id 0) (at 152.4 38.735 90))
     (property "Value" "1n" (id 1) (at 152.4 45.085 90))
-    (property "Footprint" "" (id 2) (at 152.4 41.91 0)
+    (property "Footprint" "Capacitor_SMD:C_0402_1005Metric" (id 2) (at 152.4 41.91 0)
       (effects (font (size 1.27 1.27)) hide)
     )
@@
     (property "Reference" "R401" (id 0) (at 132.715 55.245 90))
     (property "Value" "22k" (id 1) (at 132.715 59.055 90))
-    (property "Footprint" "" (id 2) (at 132.715 55.372 90)
-      (effects (font (size 1.27 1.27)) hide)
-    )
+    (property "Footprint" "Resistor_SMD:R_0402_1005Metric" (id 2) (at 132.715 55.372 90)
+      (effects (font (size 1.27 1.27)) hide)
+    )
