File: power_supply.kicad_sch (KiCad schematic)
At the start: 21 parts

Commit message: ERC valid.
Parts:
- gave numbers to parts that had none: 21
Connections:
- net SW_OUT: now reaches L101.1, U101.3 (SW)
Other:
- moved on the sheet: C104

Commit message: Assigned Footprints and Set up board specifications.
Parts:
- C100, C101: footprint (none) -> Capacitor_SMD:C_0603_1608Metric
- C102, C103, C104, C106, C108: footprint (none) -> Capacitor_SMD:C_0805_2012Metric
- C105, C107: footprint (none) -> Capacitor_SMD:C_0402_1005Metric
- D100: footprint (none) -> LED_SMD:LED_0603_1608Metric
- L100, L101: footprint (none) -> Inductor_SMD:L_0402_1005Metric
- R100: footprint (none) -> Resistor_SMD:R_0805_2012Metric
- R101, R102, R103, R104, R105: footprint (none) -> Resistor_SMD:R_0402_1005Metric
Changed lines of the file:
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@@
       (effects (font (size 1.27 1.27)) (justify left))
     )
-    (property "Footprint" "" (id 2) (at 83.82 44.45 0)
+    (property "Footprint" "Capacitor_SMD:C_0805_2012Metric" (id 2) (at 83.82 44.45 0)
       (effects (font (size 1.27 1.27)) hide)
     )
@@
       (effects (font (size 1.27 1.27)) (justify left))
     )
-    (property "Footprint" "" (id 2) (at 116.84 44.45 0)
+    (property "Footprint" "Capacitor_SMD:C_0805_2012Metric" (id 2) (at 116.84 44.45 0)
       (effects (font (size 1.27 1.27)) hide)
     )
@@
       (effects (font (size 1.27 1.27)) (justify left))
     )
-    (property "Footprint" "" (id 2) (at 33.02 43.18 0)
+    (property "Footprint" "Capacitor_SMD:C_0603_1608Metric" (id 2) (at 33.02 43.18 0)
       (effects (font (size 1.27 1.27)) hide)
     )
@@
       (effects (font (size 1.27 1.27)) (justify left))
     )
-    (property "Footprint" "" (id 2) (at 55.88 43.18 0)
+    (property "Footprint" "Capacitor_SMD:C_0603_1608Metric" (id 2) (at 55.88 43.18 0)
       (effects (font (size 1.27 1.27)) hide)
     )
@@
     (property "Reference" "L100" (id 0) (at 44.45 32.004 90))
     (property "Value" "10n" (id 1) (at 44.45 34.3154 90))
-    (property "Footprint" "" (id 2) (at 44.45 36.83 0)
+    (property "Footprint" "Inductor_SMD:L_0402_1005Metric" (id 2) (at 44.45 36.83 0)
       (effects (font (size 1.27 1.27)) hide)
     )
@@
       (effects (font (size 1.27 1.27)) (justify left))
     )
-    (property "Footprint" "" (id 2) (at 80.01 81.28 0)
+    (property "Footprint" "Capacitor_SMD:C_0805_2012Metric" (id 2) (at 80.01 81.28 0)
       (effects (font (size 1.27 1.27)) hide)
     )
@@
       (effects (font (size 1.27 1.27)) (justify left))
     )
-    (property "Footprint" "" (id 2) (at 129.54 79.375 0)
+    (property "Footprint" "Capacitor_SMD:C_0805_2012Metric" (id 2) (at 129.54 79.375 0)
       (effects (font (size 1.27 1.27)) hide)
     )
@@
       (effects (font (size 1.27 1.27)) (justify left))
     )
-    (property "Footprint" "" (id 2) (at 140.462 78.74 90)
+    (property "Footprint" "Resistor_SMD:R_0402_1005Metric" (id 2) (at 140.462 78.74 90)
       (effects (font (size 1.27 1.27)) hide)
     )
@@
       (effects (font (size 1.27 1.27)) (justify left))
     )
-    (property "Footprint" "" (id 2) (at 140.462 91.44 90)
+    (property "Footprint" "Resistor_SMD:R_0402_1005Metric" (id 2) (at 140.462 91.44 90)
       (effects (font (size 1.27 1.27)) hide)
     )
@@
       (effects (font (size 1.27 1.27)) (justify left))
     )
-    (property "Footprint" "" (id 2) (at 151.13 80.01 0)
+    (property "Footprint" "Capacitor_SMD:C_0402_1005Metric" (id 2) (at 151.13 80.01 0)
       (effects (font (size 1.27 1.27)) hide)
     )
@@
     (property "Reference" "L101" (id 0) (at 118.11 70.104 90))
     (property "Value" "68u" (id 1) (at 118.11 72.4154 90))
-    (property "Footprint" "" (id 2) (at 118.11 74.93 0)
+    (property "Footprint" "Inductor_SMD:L_0402_1005Metric" (id 2) (at 118.11 74.93 0)
       (effects (font (size 1.27 1.27)) hide)
     )
@@
     (property "Reference" "R100" (id 0) (at 76.2 31.5722 90))
     (property "Value" "10R" (id 1) (at 76.2 33.8836 90))
-    (property "Footprint" "" (id 2) (at 76.2 35.052 90)
+    (property "Footprint" "Resistor_SMD:R_0805_2012Metric" (id 2) (at 76.2 35.052 90)
       (effects (font (size 1.27 1.27)) hide)
     )
@@
       (effects (font (size 1.27 1.27)) (justify left))
     )
-    (property "Footprint" "" (id 2) (at 68.58 153.67 0)
+    (property "Footprint" "Capacitor_SMD:C_0805_2012Metric" (id 2) (at 68.58 153.67 0)
       (effects (font (size 1.27 1.27)) hide)
     )
@@
       (effects (font (size 1.27 1.27)) (justify left))
     )
-    (property "Footprint" "" (id 2) (at 56.642 142.24 90)
+    (property "Footprint" "Resistor_SMD:R_0402_1005Metric" (id 2) (at 56.642 142.24 90)
       (effects (font (size 1.27 1.27)) hide)
     )
@@
     (property "Reference" "C107" (id 0) (at 76.2063 135.4414 90))
     (property "Value" "100n" (id 1) (at 76.2063 138.2165 90))
-    (property "Footprint" "" (id 2) (at 76.2 140.97 0)
+    (property "Footprint" "Capacitor_SMD:C_0402_1005Metric" (id 2) (at 76.2 140.97 0)
       (effects (font (size 1.27 1.27)) hide)
     )
@@
       (effects (font (size 1.27 1.27)) (justify left))
     )
-    (property "Footprint" "" (id 2) (at 56.642 154.94 90)
+    (property "Footprint" "Resistor_SMD:R_0402_1005Metric" (id 2) (at 56.642 154.94 90)
       (effects (font (size 1.27 1.27)) hide)
     )
@@
     (property "Reference" "D100" (id 0) (at 164.1475 68.8045 0))
     (property "Value" "GREEN" (id 1) (at 164.1475 71.5796 0))
-    (property "Footprint" "" (id 2) (at 162.56 74.93 0)
+    (property "Footprint" "LED_SMD:LED_0603_1608Metric" (id 2) (at 162.56 74.93 0)
       (effects (font (size 1.27 1.27)) hide)
     )
@@
       (effects (font (size 1.27 1.27)) (justify left))
     )
-    (property "Footprint" "" (id 2) (at 170.942 80.01 90)
-      (effects (font (size 1.27 1.27)) hide)
-    )
+    (property "Footprint" "Resistor_SMD:R_0402_1005Metric" (id 2) (at 170.942 80.01 90)
+      (effects (font (size 1.27 1.27)) hide)
+    )
